Commit message: TESTNOTE:need additional hardware to run wifi version

File: src/go2_gazebo_sim/urdf/go2w/go2w_description_3d_lidar.xacro (robot description, xacro)
@@ -803,4 +803,56 @@
     </sensor>
   </gazebo>
+  <!-- Front camera for VLM exploration pipeline.
+       Mounted on Head_upper (~0.30m forward, 0.01m up from base),
+       pitched down ~5 deg for ground-ahead coverage.
+       1280x720, 120 deg HFOV, 10 Hz. -->
+  <link name="front_camera_link">
+    <inertial>
+      <origin xyz="0 0 0" rpy="0 0 0"/>
+      <mass value="0.001"/>
+      <inertia ixx="1e-6" ixy="0" ixz="0" iyy="1e-6" iyz="0" izz="1e-6"/>
+    </inertial>
+    <visual>
+      <origin xyz="0 0 0" rpy="0 0 0"/>
+      <geometry>
+        <box size="0.02 0.03 0.02"/>
+      </geometry>
+      <material name="camera_black">
+        <color rgba="0.1 0.1 0.1 1"/>
+      </material>
+    </visual>
+  </link>
+  <joint name="front_camera_joint" type="fixed">
+    <!-- Relative to Head_upper which is already at [0.285, 0, 0.01] from base.
+         Offset slightly forward + down with 5 deg pitch. -->
+    <origin xyz="0.015 0.0 -0.02" rpy="0 0.0873 0"/>
+    <parent link="Head_upper"/>
+    <child link="front_camera_link"/>
+  </joint>
+  <gazebo reference="front_camera_link">
+    <sensor name="front_camera" type="camera">
+      <always_on>true</always_on>
+      <update_rate>10.0</update_rate>
+      <camera>
+        <horizontal_fov>2.0944</horizontal_fov>
+        <image>
+          <width>1280</width>
+          <height>720</height>
+          <format>R8G8B8</format>
+        </image>
+        <clip>
+          <near>0.05</near>
+          <far>30.0</far>
+        </clip>
+      </camera>
+      <plugin name="gazebo_ros_front_camera" filename="libgazebo_ros_camera.so">
+        <ros>
+          <remapping>~/image_raw:=front_camera/image_raw</remapping>
+          <remapping>~/camera_info:=front_camera/camera_info</remapping>
+        </ros>
+        <frame_name>front_camera_link</frame_name>
+      </plugin>
+    </sensor>
+  </gazebo>
   <!-- Ground-truth odometry for navigation bootstrap. -->
   <gazebo>
