Commit message: newest update

File: src/go2w/go2_gazebo_sim/urdf/go2w/go2w_description_3d_lidar.xacro (robot description, xacro)
@@ -761,5 +761,11 @@
     </sensor>
   </gazebo>
-  <!-- Gazebo LiDAR stream for SLAM/local planning expecting /registered_scan. -->
+  <!-- Gazebo LiDAR stream approximating Unitree L1 4D LiDAR.
+       Real L1: 360° H x 90° V (upper hemisphere), 0.05-20m range, ~21600 pts/s.
+       Gazebo Classic gpu_ray crashes (SIGSEGV) when vertical max_angle exceeds
+       ~0.78 rad (~45°), so we cap at +42° here.  With the 13° forward tilt from
+       the livox_mid360.xacro joint, effective world-frame vertical coverage is
+       approximately -28° to +29° — enough to see walls and low ceilings.
+       Range min lowered to 0.05m (L1 near blind zone). -->
   <gazebo reference="livox_mid360">
     <sensor name="lidar_3d" type="gpu_ray">
@@ -769,5 +775,5 @@
         <scan>
           <horizontal>
-            <samples>1024</samples>
+            <samples>720</samples>
             <resolution>1</resolution>
             <min_angle>-3.14159</min_angle>
@@ -778,9 +784,9 @@
             <resolution>1</resolution>
             <min_angle>-0.261799</min_angle>
-            <max_angle>0.261799</max_angle>
+            <max_angle>0.7330</max_angle>
           </vertical>
         </scan>
         <range>
-          <min>0.2</min>
+          <min>0.05</min>
           <max>20.0</max>
           <resolution>0.01</resolution>
@@ -852,4 +858,20 @@
         </ros>
         <frame_name>front_camera_link</frame_name>
+      </plugin>
+    </sensor>
+  </gazebo>
+  <!-- Contact sensor on robot body for collision detection. -->
+  <gazebo reference="base">
+    <sensor name="base_contact" type="contact">
+      <always_on>true</always_on>
+      <update_rate>30.0</update_rate>
+      <contact>
+        <collision>base_link_fixed_joint_lump__base_collision</collision>
+      </contact>
+      <plugin name="gazebo_ros_bumper" filename="libgazebo_ros_bumper.so">
+        <ros>
+          <remapping>bumper_states:=contact_states</remapping>
+        </ros>
+        <frame_name>base_link</frame_name>
       </plugin>
     </sensor>
